File: Hardware/_restore_backup_2026-07-01T21-24-16-383/AcionamentoMotor50A.kicad_sch (KiCad schematic)
At the start: 19 parts, among them J1 Conn_01x02, J2 Conn_01x02, U4 TPS543021, U7 LM7805

Commit message: 2026_07_02
Alterações no esquemático para não usar bootstrap... e inicializaçao do roteamento
Parts:
- U4: footprint Package_TO_SOT_SMD:SOT-23-6_Handsoldering -> (none)
- U7: footprint Package_TO_SOT_THT:TO-220-3_Vertical -> Package_TO_SOT_THT:TO-220-5_P3.4x3.7mm_StaggerEven_Lead3.8mm_Vertical
Other:
- sheet PonteH: file PonteH.kicad_sch -> Braço2.kicad_sch
- sheet TensaoIsolada: file TensaoIsolada.kicad_sch -> Braço1.kicad_sch
Changed lines of the file:
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@@
 			)
 		)
-		(property "Footprint" "Package_TO_SOT_SMD:SOT-23-6_Handsoldering"
+		(property "Footprint" ""
 			(at 58.42 80.01 0)
 			(hide yes)
@@
 			)
 		)
-		(property "Footprint" "Package_TO_SOT_THT:TO-220-3_Vertical"
+		(property "Footprint" "Package_TO_SOT_THT:TO-220-5_P3.4x3.7mm_StaggerEven_Lead3.8mm_Vertical"
 			(at 52.705 125.73 0)
 			(hide yes)
@@
 	)
 	(sheet
-		(at 137.16 52.07)
-		(size 22.86 7.62)
+		(at 148.59 58.42)
+		(size 12.7 3.81)
 		(exclude_from_sim no)
 		(in_bom yes)
@@
 		)
 		(property "Sheetname" "TensaoIsolada"
-			(at 137.16 51.3584 0)
+			(at 148.59 57.7084 0)
 			(show_name no)
 			(do_not_autoplace no)
@@
 			)
 		)
-		(property "Sheetfile" "TensaoIsolada.kicad_sch"
-			(at 137.16 60.2746 0)
+		(property "Sheetfile" "Braço1.kicad_sch"
+			(at 148.59 62.8146 0)
 			(show_name no)
 			(do_not_autoplace no)
@@
 			)
 		)
-		(property "Sheetfile" "PonteH.kicad_sch"
+		(property "Sheetfile" "Braço2.kicad_sch"
 			(at 146.05 85.6746 0)
 			(show_name no)
