File: Hardware/AcionamentoMotor50A.kicad_pcb (KiCad board)
At the start: 2 copper layers, 57 parts, among them J1 Conn_01x02, J2 Conn_01x02, J3 Conn_01x02, Q1 IXFN420N10T, Q2 IXFN420N10T, Q3 IXFN420N10T, Q4 IXFN420N10T, U1 MP1923, U2 MP1923

Commit message: 2026_07_02
Alterações no esquemático para não usar bootstrap... e inicializaçao do roteamento
Parts:
- removed C_Bts1, C_Bts2: 10uF 50V, Capacitor_SMD:C_0805_2012Metric_Pad1.18x1.45mm_HandSolder
- removed C_GS1, C_GS2, C_GS3, C_GS4: 1nF 100V, Capacitor_SMD:C_0805_2012Metric_Pad1.18x1.45mm_HandSolder
- removed Cd1a1, Cd2a1: 1uF, Capacitor_SMD:C_1206_3216Metric_Pad1.33x1.80mm_HandSolder
- removed Cd1b1, Cd2b1: 100nF, Capacitor_SMD:C_0805_2012Metric_Pad1.18x1.45mm_HandSolder
- removed Dg1, Dg2, Dg3, Dg4: ES3B, Diode_SMD:D_SMA_Handsoldering
- removed J3: Conn_01x02, TerminalBlock_Phoenix:TerminalBlock_Phoenix_MKDS-1,5-2_1x02_P5.00mm_Horizontal
- removed Rg1, Rg1b1, Rg2, Rg2b1, Rg3, Rg3b1, Rg4, Rg4b1: 3R, Resistor_SMD:R_1206_3216Metric_Pad1.30x1.75mm_HandSolder
- added C1: 10uF, Capacitor_SMD:C_0805_2012Metric_Pad1.18x1.45mm_HandSolder, F.Cu at (57.0, 52.5)
- added C2: 100nF, Capacitor_SMD:C_0805_2012Metric_Pad1.18x1.45mm_HandSolder, F.Cu at (54.6, 52.7)
- added C3: 100nF, Capacitor_SMD:C_0805_2012Metric_Pad1.18x1.45mm_HandSolder, F.Cu at (60.7, 58.1)
- added C4: 100nF, Capacitor_SMD:C_0805_2012Metric_Pad1.18x1.45mm_HandSolder, F.Cu at (50.8, 68.1)
- added C5: 10uF, Capacitor_SMD:C_0805_2012Metric_Pad1.18x1.45mm_HandSolder, F.Cu at (53.2, 68.1)
- added C6: 100nF, Capacitor_SMD:C_0805_2012Metric_Pad1.18x1.45mm_HandSolder, F.Cu at (67.5, 68.1)
- added C7: 10uF, Capacitor_SMD:C_0805_2012Metric_Pad1.18x1.45mm_HandSolder, F.Cu at (69.9, 68.1)
- added COUT1: 22uF, Capacitor_SMD:C_0805_2012Metric_Pad1.18x1.45mm_HandSolder, F.Cu at (53.5, 57.9)
- added C_DIS1: 33pF, Capacitor_SMD:C_0805_2012Metric_Pad1.18x1.45mm_HandSolder, F.Cu at (-63.0, 188.6)
- added C_DIS2: 33pF, Capacitor_SMD:C_0805_2012Metric_Pad1.18x1.45mm_HandSolder, F.Cu at (-63.0, 191.7)
- added C_ENA1: 100nF, Capacitor_SMD:C_0805_2012Metric_Pad1.18x1.45mm_HandSolder, F.Cu at (-24.2, 240.2)
- added C_ENA2: 100nF, Capacitor_SMD:C_0805_2012Metric_Pad1.18x1.45mm_HandSolder, F.Cu at (44.2, 267.8)
- added C_ENA3: 100nF, Capacitor_SMD:C_0805_2012Metric_Pad1.18x1.45mm_HandSolder, F.Cu at (-120.3, 222.3)
- added C_ENA4: 100nF, Capacitor_SMD:C_0805_2012Metric_Pad1.18x1.45mm_HandSolder, F.Cu at (-23.1, 272.3)
- added C_FBVDD1: 220pF, Capacitor_SMD:C_0805_2012Metric_Pad1.18x1.45mm_HandSolder, F.Cu at (-11.4, 252.1)
- added C_FBVDD2: 220pF, Capacitor_SMD:C_0805_2012Metric_Pad1.18x1.45mm_HandSolder, F.Cu at (57.1, 279.9)
- added C_FBVDD3: 220pF, Capacitor_SMD:C_0805_2012Metric_Pad1.18x1.45mm_HandSolder, F.Cu at (-120.3, 234.4)
- added C_FBVDD4: 220pF, Capacitor_SMD:C_0805_2012Metric_Pad1.18x1.45mm_HandSolder, F.Cu at (-9.31, 284.6)
- added C_FBVEE1: 10pF, Capacitor_SMD:C_0805_2012Metric_Pad1.18x1.45mm_HandSolder, F.Cu at (-8.75, 240.0)
- added C_FBVEE2: 10pF, Capacitor_SMD:C_0805_2012Metric_Pad1.18x1.45mm_HandSolder, F.Cu at (59.2, 267.6)
- added C_FBVEE3: 10pF, Capacitor_SMD:C_0805_2012Metric_Pad1.18x1.45mm_HandSolder, F.Cu at (-115.5, 219.3)
- added C_FBVEE4: 10pF, Capacitor_SMD:C_0805_2012Metric_Pad1.18x1.45mm_HandSolder, F.Cu at (-6.64, 272.3)
- added C_IN1: 10uF, Capacitor_SMD:C_0805_2012Metric_Pad1.18x1.45mm_HandSolder, F.Cu at (-21.6, 247.2)
- added C_IN1b1: 100nF, Capacitor_SMD:C_0805_2012Metric_Pad1.18x1.45mm_HandSolder, F.Cu at (-24.0, 247.2)
- added C_IN2: 10uF, Capacitor_SMD:C_0805_2012Metric_Pad1.18x1.45mm_HandSolder, F.Cu at (46.7, 274.9)
- added C_IN2b1: 100nF, Capacitor_SMD:C_0805_2012Metric_Pad1.18x1.45mm_HandSolder, F.Cu at (44.0, 275.0)
- added C_IN3: 10uF, Capacitor_SMD:C_0805_2012Metric_Pad1.18x1.45mm_HandSolder, F.Cu at (-115.5, 231.3)
- added C_IN3b1: 100nF, Capacitor_SMD:C_0805_2012Metric_Pad1.18x1.45mm_HandSolder, F.Cu at (-46.5, 280.4)
- added C_IN4: 10uF, Capacitor_SMD:C_0805_2012Metric_Pad1.18x1.45mm_HandSolder, F.Cu at (-19.1, 281.0)
- added C_IN4b1: 100nF, Capacitor_SMD:C_0805_2012Metric_Pad1.18x1.45mm_HandSolder, F.Cu at (-22.2, 281.0)
- added C_INA1: 33pF, Capacitor_SMD:C_0805_2012Metric_Pad1.18x1.45mm_HandSolder, F.Cu at (-58.2, 197.7)
- added C_INA2: 33pF, Capacitor_SMD:C_0805_2012Metric_Pad1.18x1.45mm_HandSolder, F.Cu at (-58.2, 200.7)
- added C_INB1: 33pF, Capacitor_SMD:C_0805_2012Metric_Pad1.18x1.45mm_HandSolder, F.Cu at (-58.2, 203.7)
- added C_INB2: 33pF, Capacitor_SMD:C_0805_2012Metric_Pad1.18x1.45mm_HandSolder, F.Cu at (-58.2, 206.7)
- added C_PG1: 100nF, Capacitor_SMD:C_0805_2012Metric_Pad1.18x1.45mm_HandSolder, F.Cu at (-16.7, 239.4)
- added C_PG2: 100nF, Capacitor_SMD:C_0805_2012Metric_Pad1.18x1.45mm_HandSolder, F.Cu at (52.5, 266.7)
- added C_PG3: 100nF, Capacitor_SMD:C_0805_2012Metric_Pad1.18x1.45mm_HandSolder, F.Cu at (-110.6, 228.3)
- added C_PG4: 100nF, Capacitor_SMD:C_0805_2012Metric_Pad1.18x1.45mm_HandSolder, F.Cu at (-14.5, 271.5)
- added C_VCCI​a1: 100nF, Capacitor_SMD:C_0805_2012Metric_Pad1.18x1.45mm_HandSolder, F.Cu at (-53.4, 188.6)
- added C_VCCI​a2: 100nF, Capacitor_SMD:C_0805_2012Metric_Pad1.18x1.45mm_HandSolder, F.Cu at (-53.4, 191.7)
- added C_VCCI​b1: 1uF, Capacitor_SMD:C_0805_2012Metric_Pad1.18x1.45mm_HandSolder, F.Cu at (-53.4, 194.7)
- added C_VCCI​b2: 1uF, Capacitor_SMD:C_0805_2012Metric_Pad1.18x1.45mm_HandSolder, F.Cu at (-53.4, 197.7)
- added C_VDD1: 10uF, Capacitor_SMD:C_0805_2012Metric_Pad1.18x1.45mm_HandSolder, F.Cu at (-5.72, 245.6)
- added C_VDD1b1: 100nF, Capacitor_SMD:C_0805_2012Metric_Pad1.18x1.45mm_HandSolder, F.Cu at (-2.89, 245.5)
- added C_VDD2: 10uF, Capacitor_SMD:C_0805_2012Metric_Pad1.18x1.45mm_HandSolder, F.Cu at (62.9, 273.2)
- added C_VDD2b1: 100nF, Capacitor_SMD:C_0805_2012Metric_Pad1.18x1.45mm_HandSolder, F.Cu at (65.4, 273.1)
- added C_VDD3: 10uF, Capacitor_SMD:C_0805_2012Metric_Pad1.18x1.45mm_HandSolder, F.Cu at (-105.8, 213.3)
- added C_VDD3b1: 100nF, Capacitor_SMD:C_0805_2012Metric_Pad1.18x1.45mm_HandSolder, F.Cu at (-46.6, 311.9)
- added C_VDD4: 10uF, Capacitor_SMD:C_0805_2012Metric_Pad1.18x1.45mm_HandSolder, F.Cu at (-3.01, 277.7)
- added C_VDD4b1: 100nF, Capacitor_SMD:C_0805_2012Metric_Pad1.18x1.45mm_HandSolder, F.Cu at (-0.22, 277.7)
- added C_VDDA1: 10uF, Capacitor_SMD:C_0805_2012Metric_Pad1.18x1.45mm_HandSolder, F.Cu at (-53.4, 200.7)
- added C_VDDA2: 10uF, Capacitor_SMD:C_0805_2012Metric_Pad1.18x1.45mm_HandSolder, F.Cu at (-53.4, 203.7)
- added C_VDDA3: 10uF, Capacitor_SMD:C_0805_2012Metric_Pad1.18x1.45mm_HandSolder, F.Cu at (-53.4, 206.7)
- added C_VDDA4: 10uF, Capacitor_SMD:C_0805_2012Metric_Pad1.18x1.45mm_HandSolder, F.Cu at (-48.6, 188.6)
- added C_VDDB1: 10uF, Capacitor_SMD:C_0805_2012Metric_Pad1.18x1.45mm_HandSolder, F.Cu at (-48.6, 191.7)
- added C_VDDB2: 10uF, Capacitor_SMD:C_0805_2012Metric_Pad1.18x1.45mm_HandSolder, F.Cu at (-48.6, 194.7)
- added C_VDDB3: 10uF, Capacitor_SMD:C_0805_2012Metric_Pad1.18x1.45mm_HandSolder, F.Cu at (-48.6, 197.7)
- added C_VDDB4: 10uF, Capacitor_SMD:C_0805_2012Metric_Pad1.18x1.45mm_HandSolder, F.Cu at (-48.6, 200.7)
- added C_VDDGD1: 100nF, Capacitor_SMD:C_0805_2012Metric_Pad1.18x1.45mm_HandSolder, F.Cu at (-0.28, 245.4)
- added C_VDDGD2: 100nF, Capacitor_SMD:C_0805_2012Metric_Pad1.18x1.45mm_HandSolder, F.Cu at (67.9, 273.1)
- added C_VDDGD3: 100nF, Capacitor_SMD:C_0805_2012Metric_Pad1.18x1.45mm_HandSolder, F.Cu at (-105.8, 237.4)
- added C_VDDGD4: 100nF, Capacitor_SMD:C_0805_2012Metric_Pad1.18x1.45mm_HandSolder, F.Cu at (2.43, 277.7)
- added C_VEE1: 2,2uF, Capacitor_SMD:C_0805_2012Metric_Pad1.18x1.45mm_HandSolder, F.Cu at (-2.99, 241.0)
- added C_VEE2: 2,2uF, Capacitor_SMD:C_0805_2012Metric_Pad1.18x1.45mm_HandSolder, F.Cu at (65.5, 268.8)
- added C_VEE3: 2,2uF, Capacitor_SMD:C_0805_2012Metric_Pad1.18x1.45mm_HandSolder, F.Cu at (-101.0, 222.3)
- added C_VEE4: 2,2uF, Capacitor_SMD:C_0805_2012Metric_Pad1.18x1.45mm_HandSolder, F.Cu at (-0.16, 273.5)
- added C_VEEGD1: 6,8uF, Capacitor_SMD:C_0805_2012Metric_Pad1.18x1.45mm_HandSolder, F.Cu at (-5.57, 241.1)
- added C_VEEGD2: 6,8uF, Capacitor_SMD:C_0805_2012Metric_Pad1.18x1.45mm_HandSolder, F.Cu at (62.9, 268.8)
- added C_VEEGD3: 6,8uF, Capacitor_SMD:C_0805_2012Metric_Pad1.18x1.45mm_HandSolder, F.Cu at (-101.0, 234.4)
- added C_VEEGD4: 6,8uF, Capacitor_SMD:C_0805_2012Metric_Pad1.18x1.45mm_HandSolder, F.Cu at (-2.95, 273.5)
- added L1: 12uH, Inductor_SMD:L_0805_2012Metric_Pad1.05x1.20mm_HandSolder, F.Cu at (53.5, 55.7)
- added LBB1: 3,3uH, Inductor_SMD:L_0805_2012Metric_Pad1.05x1.20mm_HandSolder, F.Cu at (-7.22, 248.4)
- added LBB2: 3,3uH, Inductor_SMD:L_0805_2012Metric_Pad1.05x1.20mm_HandSolder, F.Cu at (61.4, 276.4)
- added LBB3: 3,3uH, Inductor_SMD:L_0805_2012Metric_Pad1.05x1.20mm_HandSolder, F.Cu at (-101.2, 248.5)
- added LBB4: 3,3uH, Inductor_SMD:L_0805_2012Metric_Pad1.05x1.20mm_HandSolder, F.Cu at (-5.26, 280.8)
- added R1: 470K, Resistor_SMD:R_0805_2012Metric_Pad1.20x1.40mm_HandSolder, F.Cu at (60.3, 60.5)
- added R2: 27K, Resistor_SMD:R_0805_2012Metric_Pad1.20x1.40mm_HandSolder, F.Cu at (64.4, 59.3)
- added R3: 1k, Resistor_SMD:R_0805_2012Metric_Pad1.20x1.40mm_HandSolder, F.Cu at (-86.4, 264.4)
- added R4: 100K, Resistor_SMD:R_0805_2012Metric_Pad1.20x1.40mm_HandSolder, F.Cu at (60.7, 51.9)
- added R5: 3K4, Resistor_SMD:R_0805_2012Metric_Pad1.20x1.40mm_HandSolder, F.Cu at (64.8, 55.1)
- added R6: 51k, Resistor_SMD:R_0805_2012Metric_Pad1.20x1.40mm_HandSolder, F.Cu at (-92.6, 258.6)
- added R7: 1k, Resistor_SMD:R_0805_2012Metric_Pad1.20x1.40mm_HandSolder, F.Cu at (-95.8, 257.4)
- added R8: 10k, Resistor_SMD:R_0805_2012Metric_Pad1.20x1.40mm_HandSolder, F.Cu at (-99.7, 264.1)
- added R_DT1: 20K, Resistor_SMD:R_0805_2012Metric_Pad1.20x1.40mm_HandSolder, F.Cu at (-60.5, 164.9)
- added R_DT2: 20K, Resistor_SMD:R_0805_2012Metric_Pad1.20x1.40mm_HandSolder, F.Cu at (-60.5, 167.9)
- added R_ENA1: 5K1, Resistor_SMD:R_0805_2012Metric_Pad1.20x1.40mm_HandSolder, F.Cu at (-21.0, 239.3)
- added R_ENA2: 5K1, Resistor_SMD:R_0805_2012Metric_Pad1.20x1.40mm_HandSolder, F.Cu at (47.3, 266.8)
- added R_ENA3: 5K1, Resistor_SMD:R_0805_2012Metric_Pad1.20x1.40mm_HandSolder, F.Cu at (-120.3, 249.2)
- added R_ENA4: 5K1, Resistor_SMD:R_0805_2012Metric_Pad1.20x1.40mm_HandSolder, F.Cu at (-19.6, 271.4)
- added R_FBVDDBOT1: 10K, Resistor_SMD:R_0805_2012Metric_Pad1.20x1.40mm_HandSolder, F.Cu at (-11.5, 249.7)
- added R_FBVDDBOT2: 10K, Resistor_SMD:R_0805_2012Metric_Pad1.20x1.40mm_HandSolder, F.Cu at (57.2, 277.7)
- added R_FBVDDBOT3: 10K, Resistor_SMD:R_0805_2012Metric_Pad1.20x1.40mm_HandSolder, F.Cu at (-115.5, 246.2)
- added R_FBVDDBOT4: 10K, Resistor_SMD:R_0805_2012Metric_Pad1.20x1.40mm_HandSolder, F.Cu at (-9.29, 282.2)
- added R_FBVDDTOP1: 50K, Resistor_SMD:R_0805_2012Metric_Pad1.20x1.40mm_HandSolder, F.Cu at (-11.4, 254.4)
- added R_FBVDDTOP2: 50K, Resistor_SMD:R_0805_2012Metric_Pad1.20x1.40mm_HandSolder, F.Cu at (57.2, 282.3)
- added R_FBVDDTOP3: 50K, Resistor_SMD:R_0805_2012Metric_Pad1.20x1.40mm_HandSolder, F.Cu at (-57.0, 245.7)
- added R_FBVDDTOP4: 50K, Resistor_SMD:R_0805_2012Metric_Pad1.20x1.40mm_HandSolder, F.Cu at (-9.21, 287.1)
- added R_FBVEE1: 55K, Resistor_SMD:R_0805_2012Metric_Pad1.20x1.40mm_HandSolder, F.Cu at (-0.54, 240.9)
- added R_FBVEE2: 55K, Resistor_SMD:R_0805_2012Metric_Pad1.20x1.40mm_HandSolder, F.Cu at (67.7, 268.9)
- added R_FBVEE3: 55K, Resistor_SMD:R_0805_2012Metric_Pad1.20x1.40mm_HandSolder, F.Cu at (-102.0, 243.2)
- added R_FBVEE4: 55K, Resistor_SMD:R_0805_2012Metric_Pad1.20x1.40mm_HandSolder, F.Cu at (2.44, 273.4)
- added R_G1: 10R, Resistor_SMD:R_0805_2012Metric_Pad1.20x1.40mm_HandSolder, F.Cu at (-60.5, 170.8)
- added R_G2: 10R, Resistor_SMD:R_0805_2012Metric_Pad1.20x1.40mm_HandSolder, F.Cu at (-60.5, 173.8)
- added R_G3: 10R, Resistor_SMD:R_0805_2012Metric_Pad1.20x1.40mm_HandSolder, F.Cu at (-60.5, 176.7)
- added R_G4: 10R, Resistor_SMD:R_0805_2012Metric_Pad1.20x1.40mm_HandSolder, F.Cu at (-55.8, 164.9)
- added R_GS1: 10K, Resistor_SMD:R_0805_2012Metric_Pad1.20x1.40mm_HandSolder, F.Cu at (-55.8, 167.9)
- added R_GS2: 10K, Resistor_SMD:R_0805_2012Metric_Pad1.20x1.40mm_HandSolder, F.Cu at (-55.8, 170.8)
- added R_GS3: 10K, Resistor_SMD:R_0805_2012Metric_Pad1.20x1.40mm_HandSolder, F.Cu at (-55.8, 173.8)
- added R_GS4: 10K, Resistor_SMD:R_0805_2012Metric_Pad1.20x1.40mm_HandSolder, F.Cu at (-55.8, 176.7)
- added R_INA1: 51R, Resistor_SMD:R_0805_2012Metric_Pad1.20x1.40mm_HandSolder, F.Cu at (-51.0, 164.9)
- added R_INA2: 51R, Resistor_SMD:R_0805_2012Metric_Pad1.20x1.40mm_HandSolder, F.Cu at (-51.0, 167.9)
- added R_INB1: 51R, Resistor_SMD:R_0805_2012Metric_Pad1.20x1.40mm_HandSolder, F.Cu at (-51.0, 170.8)
- added R_INB2: 51R, Resistor_SMD:R_0805_2012Metric_Pad1.20x1.40mm_HandSolder, F.Cu at (-51.0, 173.8)
- added R_PG1: 5K1, Resistor_SMD:R_0805_2012Metric_Pad1.20x1.40mm_HandSolder, F.Cu at (-18.8, 239.3)
- added R_PG2: 5K1, Resistor_SMD:R_0805_2012Metric_Pad1.20x1.40mm_HandSolder, F.Cu at (49.9, 266.8)
- added R_PG3: 5K1, Resistor_SMD:R_0805_2012Metric_Pad1.20x1.40mm_HandSolder, F.Cu at (-106.0, 252.1)
- added R_PG4: 5K1, Resistor_SMD:R_0805_2012Metric_Pad1.20x1.40mm_HandSolder, F.Cu at (-17.2, 271.4)
- added R_Sh1: 0.001R, Resistor_THT:R_Axial_Power_L20.0mm_W6.4mm_P25.40mm, F.Cu at (-92.8, 191.1)
- added U3: UCC34141-Q1, ZeniteSolar:SSOP-16_4.55x10.63mm_P0.65mm, F.Cu at (50.8, 269.9)
- added U4: TPS543021, Package_TO_SOT_SMD:SOT-23-6_Handsoldering, F.Cu at (60.6, 55.1)
- added U5: UCC34141-Q1, ZeniteSolar:SSOP-16_4.55x10.63mm_P0.65mm, F.Cu at (-15.9, 274.5)
- added U6: UCC34141-Q1, ZeniteSolar:SSOP-16_4.55x10.63mm_P0.65mm, F.Cu at (-77.6, 242.7)
- added U7: LM7805, Package_TO_SOT_THT:TO-220-3_Vertical, F.Cu at (58.1, 66.9)
- added U8: UCC21550, Package_SO:SOIC-16W_7.5x10.3mm_P1.27mm, F.Cu at (-56.5, 120.7)
- added U9: Opamp_Quad, Package_SO:SOIC-14_3.9x8.7mm_P1.27mm, F.Cu at (-93.2, 264.4)
- A1: moved to B.Cu
- U1: value MP1923 -> UCC21550; footprint Package_SO:SOP-8_3.76x4.96mm_P1.27mm -> Package_SO:SOIC-16W_7.5x10.3mm_P1.27mm
- U2: value MP1923 -> UCC34141-Q1; footprint Package_SO:SOP-8_3.76x4.96mm_P1.27mm -> ZeniteSolar:SSOP-16_4.55x10.63mm_P0.65mm
- moved RSnb1a1 321.0 mm to (-92.8, 139.7)
- moved RSnb1ab1 321.0 mm to (-92.8, 150.2)
- moved RSnb2 321.0 mm to (-92.8, 108.0)
- moved RSnb2b1 321.0 mm to (-92.8, 160.8)
- moved RSnb3 321.0 mm to (-92.8, 118.6)
- moved RSnb3b1 321.0 mm to (-92.8, 171.3)
- moved RSnb4 321.0 mm to (-92.8, 129.1)
- moved RSnb4b1 321.0 mm to (-92.8, 181.9)
- moved HS1 306.4 mm to (-117.4, 5.38)
- moved Q1 262.6 mm to (-219.0, 112.6)
- moved C_DS3a1 259.1 mm to (-63.0, 206.7)
- moved Q3 257.4 mm to (-213.8, 168.3)
- moved C_DS1a1 250.3 mm to (-63.0, 194.7)
- moved C_DS1b1 250.3 mm to (-63.0, 197.7)
- moved C_DS2a1 250.3 mm to (-63.0, 200.7)
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Connections:
- net +60V renamed BAT+
- A1 pad 20: Net-(A1-D5) -> PWM1
- A1 pad 21: Net-(A1-D6) -> PWM2
- A1 pad 24: Net-(A1-D9) -> PWM3
- A1 pad 25: Net-(A1-D10) -> PWM4
- A1 pad 29: GNDREF -> BAT-
- A1 pad 4: unconnected-(A1-3V3-Pad4) -> 3v3
- A1 pad 6: GNDREF -> BAT-
- A1 pad 7: GNDREF -> BAT-
- CSnb2 pad 2: GNDREF -> BAT-
- CSnb4 pad 2: GNDREF -> BAT-
- C_DS2a1 pad 2: GNDREF -> BAT-
- C_DS2b1 pad 2: GNDREF -> BAT-
- C_DS4a1 pad 2: GNDREF -> BAT-
- C_DS4b1 pad 2: GNDREF -> BAT-
- J1 pad 1: +12V -> +24V
- J1 pad 2: GNDREF -> BAT-
- J2 pad 2: GNDREF -> BAT-
- Q1 pad 1: G_SW1 -> GATE1
- Q2 pad 1: G_SW2 -> GATE2
- Q2 pad 2: GNDREF -> Vsh
- Q2 pad 3: GNDREF -> Vsh
- Q3 pad 1: G_SW3 -> GATE3
- Q4 pad 1: G_SW4 -> GATE4
- Q4 pad 2: GNDREF -> Vsh
- Q4 pad 3: GNDREF -> Vsh
- U1 pad 1: +12V -> INA1
- U1 pad 2: BTS1 -> INB1
- U1 pad 3: Net-(U1-DRVH) -> +5V
- U1 pad 4: VA -> BAT-
- U1 pad 5: Net-(A1-D10) -> DIS1
- U1 pad 6: Net-(A1-D9) -> DT1
- U1 pad 7: GNDREF -> unconnected-(U1-NC-Pad7)
- U1 pad 8: Net-(U1-DRVL) -> +5V
- U2 pad 1: +12V -> ENA
- U2 pad 2: BTS2 -> PG
- U2 pad 3: Net-(U2-DRVH) -> +18V
- U2 pad 4: VB -> +18V
- U2 pad 5: Net-(A1-D6) -> BAT-
- U2 pad 6: Net-(A1-D5) -> BAT-
- U2 pad 7: GNDREF -> BAT-
- U2 pad 8: Net-(U2-DRVL) -> BAT-
Routing:
- net BAT-: track 0.00 -> 154.1 mm, vias 0 -> 3
- net +18V: track 0.00 -> 47.7 mm, vias 0 -> 1
- net COMA2: track 0.00 -> 39.6 mm, vias 0 -> 2
- net COMA: track 0.00 -> 38.8 mm, vias 0 -> 2
- net +24V: track 0.00 -> 29.2 mm, vias 0 -> 2
- net +15v_ISO1: track 0.00 -> 27.3 mm
- net +15v_ISO2: track 0.00 -> 26.7 mm
- net FBVEE: track 0.00 -> 16.9 mm
- net FBVEE2: track 0.00 -> 16.6 mm
- net FBVDD2: track 0.00 -> 12.9 mm
- net FBVDD: track 0.00 -> 12.8 mm
- net +5V: track 0.00 -> 12.5 mm, vias 0 -> 1
- net Net-(U9A--): track 0.00 -> 9.69 mm
- net Net-(U9B--): track 0.00 -> 9.68 mm
- net Net-(U4-SW): track 0.00 -> 9.08 mm, vias 0 -> 2
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
Commit message: roteamento de fonte isolada
Parts:
- moved Q4 149.7 mm to (-241.5, 280.6)
- moved C_VDD3b1 68.7 mm to (-60.7, 244.6), turned to -90 degrees
- moved C_FBVDD3 65.9 mm to (-54.5, 238.9), turned to 180 degrees
- moved R_FBVDDBOT3 61.7 mm to (-54.6, 236.3), turned to 180 degrees
- moved C_FBVEE3 57.6 mm to (-59.1, 231.3)
- moved C_VDD3 52.7 mm to (-63.4, 244.6), turned to -90 degrees
- moved C_ENA3 50.7 mm to (-71.8, 237.5), turned to 180 degrees
- moved R_ENA3 50.4 mm to (-71.8, 235.3)
- moved C_VDDGD3 48.3 mm to (-58.1, 244.7), turned to -90 degrees
- moved R_FBVEE3 44.8 mm to (-58.1, 234.5), turned to 90 degrees
- moved C_PG3 41.1 mm to (-71.8, 241.9), turned to 180 degrees
- moved C_VEEGD3 40.7 mm to (-60.3, 234.5), turned to 90 degrees
- moved C_VEE3 40.2 mm to (-62.7, 234.5), turned to 90 degrees
- moved LBB3 38.9 mm to (-64.9, 234.5), turned to -90 degrees
- moved R_PG3 36.4 mm to (-71.8, 239.7)
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Routing:
- net COMA3: track 0.00 -> 49.4 mm
- net +15v_ISO3: track 0.00 -> 16.1 mm
- net -5v_ISO3: track 0.00 -> 9.19 mm
- net BSW3: track 0.00 -> 8.36 mm
- net FBVDD3: track 0.00 -> 8.30 mm
- net FBVEE3: track 0.00 -> 7.06 mm

Commit message: 2026_07_03
Continuidade do roteamento..

foram roteados os drivers
Parts:
- moved C_IN3 249.3 mm to (82.4, 79.7), turned to 90 degrees
- moved C_VDDA2 244.9 mm to (130.5, 42.0), turned to -90 degrees
- moved C_VDDA1 244.7 mm to (132.9, 42.0), turned to -90 degrees
- moved R_FBVDDTOP1 243.4 mm to (99.3, 37.7)
- moved LBB1 243.3 mm to (91.9, 26.2), turned to 90 degrees
- moved C_FBVDD1 243.3 mm to (99.4, 35.5)
- moved R_FBVDDBOT1 243.3 mm to (99.3, 33.2)
- moved C_IN3b1 239.8 mm to (84.6, 79.6), turned to 90 degrees
- moved C_INA1 238.4 mm to (118.0, 37.2), turned to 90 degrees
- moved C_INB1 237.6 mm to (114.2, 40.3), turned to 180 degrees
- moved C_FBVEE1 236.6 mm to (95.0, 27.4), turned to 0 degrees
- moved R_G1 235.3 mm to (134.3, 38.9)
- moved C_IN1b1 233.3 mm to (81.4, 39.2)
- moved C_IN1 233.3 mm to (83.9, 39.2)
- moved U2 233.1 mm to (86.2, 33.5)
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Connections:
- C_VEE4 pad 2: COMA -> COMA4
- C_VEEGD4 pad 2: COMA -> COMA4
- LBB4 pad 1: COMA -> COMA4
Routing:
- net BAT-: track 154.1 -> 239.6 mm
- net +18V: track 47.7 -> 107.2 mm, vias 1 -> 2
- net COMA4: track 0.00 -> 41.0 mm
- net +5V: track 12.5 -> 46.3 mm, vias 1 -> 0
- net BSW4: track 0.00 -> 14.9 mm
- net +15v_ISO1: track 27.3 -> 12.9 mm
- net +15v_ISO2: track 26.7 -> 13.9 mm
- net +15v_ISO4: track 0.00 -> 12.2 mm
- net OUTA2: track 0.00 -> 11.9 mm
- net OUTA1: track 0.00 -> 11.7 mm
- net DIS1: track 0.00 -> 10.7 mm
- net OUTB2: track 0.00 -> 9.32 mm
- net -5v_ISO4: track 0.00 -> 9.12 mm
- net BSW2: track 5.40 -> 14.4 mm
- net VSSB2: track 0.00 -> 8.85 mm
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
Commit message: 2026_07_04
Todas as ligações foram feitas.

Faltar rodar DRC
Verificar as regras JLPCB
Parts:
- removed HS1: Heatsink, ZeniteSolar:Heatsink_120mmx100mm_H70mm
- added C8: 100nF, Capacitor_SMD:C_0805_2012Metric_Pad1.18x1.45mm_HandSolder, F.Cu at (201.3, 161.9)
- added C9: 10uF, Capacitor_SMD:C_0805_2012Metric_Pad1.18x1.45mm_HandSolder, F.Cu at (199.0, 161.8)
- C_DS1a1, C_DS1b1, C_DS2a1, C_DS2b1, DSnb1, DSnb2, Q1, Q2, Q3, Q4: moved to B.Cu
- moved Q4 549.2 mm to (294.8, 162.2), turned to 90 degrees
- moved Q3 512.6 mm to (295.3, 107.7), turned to 90 degrees
- moved Q1 484.8 mm to (265.8, 107.9), turned to 90 degrees
- moved Q2 470.4 mm to (265.5, 161.8), turned to 90 degrees
- moved RSnb4b1 425.9 mm to (331.7, 147.2), turned to -90 degrees
- moved RSnb3b1 422.8 mm to (326.3, 115.9), turned to 90 degrees
- moved RSnb4 403.5 mm to (310.3, 146.8), turned to -90 degrees
- moved RSnb3 401.5 mm to (308.7, 116.0), turned to 90 degrees
- moved C_DS3a1 397.9 mm to (318.1, 92.4), turned to 180 degrees
- moved CSnb4 386.4 mm to (323.7, 174.6), turned to 90 degrees
- moved CSnb3 379.8 mm to (317.1, 106.7), turned to 90 degrees
- moved DSnb3 377.5 mm to (317.1, 112.9), turned to -90 degrees
- moved DSnb4 375.8 mm to (318.0, 162.2), turned to 90 degrees
- moved R_Sh1 366.5 mm to (273.6, 186.7), turned to 90 degrees
- moved C_DS2b1 352.1 mm to (225.9, 157.1)
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Connections:
- R_G2 pad 2: GATE2 -> GATE3
- R_G4 pad 2: GATE3 -> GATE2
- R_GS2 pad 2: GATE2 -> GATE3
- R_GS4 pad 2: GATE3 -> GATE2
Routing:
- net BAT+: track 0.00 -> 491.8 mm
- net BAT-: track 239.6 -> 622.2 mm, vias 3 -> 13
- net VB: track 0.00 -> 233.0 mm
- net VA: track 0.00 -> 218.9 mm
- net Vsh: track 0.00 -> 145.5 mm, vias 0 -> 2
- net GATE3: track 2.32 -> 87.5 mm
- net GATE4: track 2.65 -> 85.7 mm
- net PWM3: track 0.00 -> 73.5 mm
- net PWM4: track 0.00 -> 73.5 mm
- net Net-(DSnb3-K): track 0.00 -> 72.9 mm
- net +18V: track 107.2 -> 176.7 mm, vias 2 -> 7
- net PWM1: track 0.00 -> 68.8 mm
- net 3v3: track 0.00 -> 68.8 mm
- net PWM2: track 0.00 -> 62.5 mm, vias 0 -> 2
- net DIS1: track 10.7 -> 69.6 mm, vias 0 -> 4
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- added copper zone on F.Cu, net +5V
- added copper zone on B.Cu, net BAT-
Other:
- board outline added: 265 x 150 mm

Commit message: Ajustes do DRC. Removida a solder mask das trilhas de potência.
Parts:
- moved C_VEE4 0.80 mm to (169.7, 151.5)
- moved C_VEE3 0.78 mm to (167.9, 129.2)
- moved C_VEEGD1 0.66 mm to (167.9, 88.1)
- moved C_VEEGD3 0.48 mm to (170.6, 129.1)
- moved C_VEEGD2 0.45 mm to (167.6, 107.9)
- moved R_ENA2 0.39 mm to (157.9, 108.1)
- moved C_VEE1 0.34 mm to (170.4, 88.2)
- moved C_ENA3 0.34 mm to (161.3, 133.5)
- moved C_IN3b1 0.30 mm to (161.3, 137.5)
- moved C_VEEGD4 0.30 mm to (172.5, 151.5)
- moved C_IN3 0.23 mm to (159.1, 137.5)
- moved C_PG3 0.12 mm to (163.8, 129.0)
Routing:
- net 3v3: track 68.8 -> 71.8 mm
- net BAT-: track 622.2 -> 619.3 mm
- net COMA4: track 41.0 -> 43.0 mm
- net BAT+: track 491.8 -> 493.8 mm
- net BSW3: track 14.9 -> 16.8 mm
- net GATE3: track 87.5 -> 85.7 mm
- net BSW: track 14.2 -> 16.0 mm
- net COMA3: track 43.8 -> 45.5 mm
- net VDDA2: track 7.16 -> 5.63 mm
- net VDDB2: track 7.13 -> 5.64 mm
- net BSW4: track 14.9 -> 16.3 mm
- net COMA: track 45.3 -> 46.6 mm
- net BSW2: track 14.4 -> 15.7 mm
- net FBVEE2: track 8.46 -> 9.56 mm
- net PG4: track 8.79 -> 7.69 mm
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
Commit message: 2026_07_05
PCB Finalizada
Parts:
- moved R_DT1 3.65 mm to (189.9, 110.4), turned to 0 degrees
Routing:
- net BAT-: track 619.3 -> 569.1 mm, vias 13 -> 16
- net +5V: track 102.4 -> 115.9 mm, vias 18 -> 24
- net PWM2: track 62.5 -> 59.5 mm, vias 2 -> 0
- net PWM1: track 68.8 -> 65.9 mm
- net COMA: track 46.6 -> 44.5 mm
- net PG2: track 7.28 -> 6.36 mm
- net BSW: track 16.0 -> 15.1 mm
- net DT1: track 7.35 -> 6.57 mm
- net ENA2: track 6.63 -> 5.84 mm
- net DIS1: track 69.5 -> 69.2 mm, vias 4 -> 2
- net VB: vias 0 -> 1
- net VA: vias 0 -> 1

Commit message: 2026_07_22
Finalizada a PCB para fazer na fresa do IFSC
Parts:
- removed C4, C6, C_ENA1, C_ENA2, C_ENA3, C_ENA4, C_IN1b1, C_IN2b1, C_IN3b1, C_IN4b1, C_PG1, C_PG2, C_PG3, C_PG4, C_VDD1b1, C_VDD2b1, C_VDD3b1, C_VDD4b1, C_VDDGD1, C_VDDGD2, C_VDDGD3, C_VDDGD4: 100nF, Capacitor_SMD:C_0805_2012Metric_Pad1.18x1.45mm_HandSolder
- removed C5, C7, C_IN1, C_IN2, C_IN3, C_IN4, C_VDD1, C_VDD2, C_VDD3, C_VDD4: 10uF, Capacitor_SMD:C_0805_2012Metric_Pad1.18x1.45mm_HandSolder
- removed C_FBVDD1, C_FBVDD2, C_FBVDD3, C_FBVDD4: 220pF, Capacitor_SMD:C_0805_2012Metric_Pad1.18x1.45mm_HandSolder
- removed C_FBVEE1, C_FBVEE2, C_FBVEE3, C_FBVEE4: 10pF, Capacitor_SMD:C_0805_2012Metric_Pad1.18x1.45mm_HandSolder
- removed C_VEE1, C_VEE2, C_VEE3, C_VEE4: 2,2uF, Capacitor_SMD:C_0805_2012Metric_Pad1.18x1.45mm_HandSolder
- removed C_VEEGD1, C_VEEGD2, C_VEEGD3, C_VEEGD4: 6,8uF, Capacitor_SMD:C_0805_2012Metric_Pad1.18x1.45mm_HandSolder
- removed LBB1, LBB2, LBB3, LBB4: 3,3uH, Inductor_SMD:L_0805_2012Metric_Pad1.05x1.20mm_HandSolder
- removed R7: 1k, Resistor_SMD:R_0805_2012Metric_Pad1.20x1.40mm_HandSolder
- removed R8: 10k, Resistor_SMD:R_0805_2012Metric_Pad1.20x1.40mm_HandSolder
- removed R_ENA1, R_ENA2, R_ENA3, R_ENA4, R_PG1, R_PG2, R_PG3, R_PG4: 5K1, Resistor_SMD:R_0805_2012Metric_Pad1.20x1.40mm_HandSolder
- removed R_FBVDDBOT1, R_FBVDDBOT2, R_FBVDDBOT3, R_FBVDDBOT4: 10K, Resistor_SMD:R_0805_2012Metric_Pad1.20x1.40mm_HandSolder
- removed R_FBVDDTOP1, R_FBVDDTOP2, R_FBVDDTOP3, R_FBVDDTOP4: 50K, Resistor_SMD:R_0805_2012Metric_Pad1.20x1.40mm_HandSolder
- removed R_FBVEE1, R_FBVEE2, R_FBVEE3, R_FBVEE4: 55K, Resistor_SMD:R_0805_2012Metric_Pad1.20x1.40mm_HandSolder
- removed R_Sh1: 0.001R, Resistor_THT:R_Axial_Power_L20.0mm_W6.4mm_P25.40mm
- removed U2, U3, U5, U6: UCC34141-Q1, ZeniteSolar:SSOP-16_4.55x10.63mm_P0.65mm
- added CFBVDD_1: 330pF, Capacitor_SMD:C_0805_2012Metric_Pad1.18x1.45mm_HandSolder, F.Cu at (167.8, 66.9)
- added CFBVDD_2: 330pF, Capacitor_SMD:C_0805_2012Metric_Pad1.18x1.45mm_HandSolder, F.Cu at (167.6, 96.7)
- added CFBVDD_3: 330pF, Capacitor_SMD:C_0805_2012Metric_Pad1.18x1.45mm_HandSolder, F.Cu at (167.5, 119.8)
- added CFBVDD_4: 330pF, Capacitor_SMD:C_0805_2012Metric_Pad1.18x1.45mm_HandSolder, F.Cu at (167.3, 155.2)
- added CFBVEE_1: 330pF, Capacitor_SMD:C_0805_2012Metric_Pad1.18x1.45mm_HandSolder, F.Cu at (171.5, 71.0)
- added CFBVEE_2: 330pF, Capacitor_SMD:C_0805_2012Metric_Pad1.18x1.45mm_HandSolder, F.Cu at (172.0, 98.0)
- added CFBVEE_3: 330pF, Capacitor_SMD:C_0805_2012Metric_Pad1.18x1.45mm_HandSolder, F.Cu at (171.4, 124.4)
- added CFBVEE_4: 330pF, Capacitor_SMD:C_0805_2012Metric_Pad1.18x1.45mm_HandSolder, F.Cu at (171.7, 158.6)
- added COUT2: 100nF, Capacitor_SMD:C_0805_2012Metric_Pad1.18x1.45mm_HandSolder, F.Cu at (128.2, 74.4)
- added Cin1: 20uF, Capacitor_SMD:C_0805_2012Metric_Pad1.18x1.45mm_HandSolder, F.Cu at (150.4, 75.4)
- added Cin1b1: 100nF, Capacitor_SMD:C_0805_2012Metric_Pad1.18x1.45mm_HandSolder, F.Cu at (152.8, 75.4)
- added Cin2: 20uF, Capacitor_SMD:C_0805_2012Metric_Pad1.18x1.45mm_HandSolder, F.Cu at (153.6, 103.4)
- added Cin2b1: 100nF, Capacitor_SMD:C_0805_2012Metric_Pad1.18x1.45mm_HandSolder, F.Cu at (150.8, 103.4)
- added Cin3: 20uF, Capacitor_SMD:C_0805_2012Metric_Pad1.18x1.45mm_HandSolder, F.Cu at (153.4, 129.3)
- added Cin3b1: 100nF, Capacitor_SMD:C_0805_2012Metric_Pad1.18x1.45mm_HandSolder, F.Cu at (150.8, 129.3)
- added Cin4: 20uF, Capacitor_SMD:C_0805_2012Metric_Pad1.18x1.45mm_HandSolder, F.Cu at (153.2, 162.3)
- added Cin4b1: 100nF, Capacitor_SMD:C_0805_2012Metric_Pad1.18x1.45mm_HandSolder, F.Cu at (150.6, 162.3)
- added Cout1a1: 100nF, Capacitor_SMD:C_0805_2012Metric_Pad1.18x1.45mm_HandSolder, F.Cu at (169.8, 80.5)
- added Cout1b1: 10uF, Capacitor_SMD:C_0805_2012Metric_Pad1.18x1.45mm_HandSolder, F.Cu at (172.1, 80.5)
- added Cout1c1: 10uF, Capacitor_SMD:C_0805_2012Metric_Pad1.18x1.45mm_HandSolder, F.Cu at (174.5, 80.5)
- added Cout2_1: 4.7uF, Capacitor_SMD:C_0805_2012Metric_Pad1.18x1.45mm_HandSolder, F.Cu at (177.9, 81.4)
- added Cout2_2: 4.7uF, Capacitor_SMD:C_0805_2012Metric_Pad1.18x1.45mm_HandSolder, F.Cu at (176.8, 108.2)
- added Cout2_3: 4.7uF, Capacitor_SMD:C_0805_2012Metric_Pad1.18x1.45mm_HandSolder, F.Cu at (177.6, 134.7)
- added Cout2_4: 4.7uF, Capacitor_SMD:C_0805_2012Metric_Pad1.18x1.45mm_HandSolder, F.Cu at (176.9, 167.0)
- added Cout2a1: 100nF, Capacitor_SMD:C_0805_2012Metric_Pad1.18x1.45mm_HandSolder, F.Cu at (174.4, 108.3)
- added Cout2b1: 10uF, Capacitor_SMD:C_0805_2012Metric_Pad1.18x1.45mm_HandSolder, F.Cu at (172.0, 108.2)
- added Cout2c1: 10uF, Capacitor_SMD:C_0805_2012Metric_Pad1.18x1.45mm_HandSolder, F.Cu at (169.8, 108.2)
- added Cout3_1: 12uF, Capacitor_SMD:C_0805_2012Metric_Pad1.18x1.45mm_HandSolder, F.Cu at (178.3, 72.8)
- added Cout3_2: 12uF, Capacitor_SMD:C_0805_2012Metric_Pad1.18x1.45mm_HandSolder, F.Cu at (176.0, 101.1)
- added Cout3_3: 12uF, Capacitor_SMD:C_0805_2012Metric_Pad1.18x1.45mm_HandSolder, F.Cu at (178.5, 126.3)
- added Cout3_4: 12uF, Capacitor_SMD:C_0805_2012Metric_Pad1.18x1.45mm_HandSolder, F.Cu at (176.0, 159.6)
- added Cout3a1: 100nF, Capacitor_SMD:C_0805_2012Metric_Pad1.18x1.45mm_HandSolder, F.Cu at (174.3, 133.8)
- added Cout3b1: 10uF, Capacitor_SMD:C_0805_2012Metric_Pad1.18x1.45mm_HandSolder, F.Cu at (171.9, 133.9)
- added Cout3c1: 10uF, Capacitor_SMD:C_0805_2012Metric_Pad1.18x1.45mm_HandSolder, F.Cu at (169.6, 133.8)
- added Cout4a1: 100nF, Capacitor_SMD:C_0805_2012Metric_Pad1.18x1.45mm_HandSolder, F.Cu at (174.5, 167.0)
- added Cout4b1: 10uF, Capacitor_SMD:C_0805_2012Metric_Pad1.18x1.45mm_HandSolder, F.Cu at (172.2, 167.1)
- added Cout4c1: 10uF, Capacitor_SMD:C_0805_2012Metric_Pad1.18x1.45mm_HandSolder, F.Cu at (169.8, 167.1)
- added D1: 1N4148, Diode_THT:D_DO-35_SOD27_P7.62mm_Horizontal, B.Cu at (171.3, 76.3)
- added D2: 1N4148, Diode_THT:D_DO-35_SOD27_P7.62mm_Horizontal, B.Cu at (171.2, 104.6)
- added D3: 1N4148, Diode_THT:D_DO-35_SOD27_P7.62mm_Horizontal, B.Cu at (171.3, 130.1)
- added D4: 1N4148, Diode_THT:D_DO-35_SOD27_P7.62mm_Horizontal, B.Cu at (170.9, 163.4)
- added HO100P1: Conn_01x05, Connector_Molex:Molex_KK-254_AE-6410-05A_1x05_P2.54mm_Vertical, F.Cu at (141.7, 176.3)
- added HS1: Heatsink, ZeniteSolar:Heatsink_120mmx100mm_H70mm, B.Cu at (267.5, 123.2)
- added RFBVDD_VDD1: 90K, Resistor_SMD:R_0805_2012Metric_Pad1.20x1.40mm_HandSolder, F.Cu at (172.2, 67.7)
- added RFBVDD_VDD2: 90K, Resistor_SMD:R_0805_2012Metric_Pad1.20x1.40mm_HandSolder, F.Cu at (172.0, 95.9)
- added RFBVDD_VDD3: 90K, Resistor_SMD:R_0805_2012Metric_Pad1.20x1.40mm_HandSolder, F.Cu at (171.8, 121.0)
- added RFBVDD_VDD4: 90K, Resistor_SMD:R_0805_2012Metric_Pad1.20x1.40mm_HandSolder, F.Cu at (171.3, 154.0)
- added RFBVDD_VEE1: 10K, Resistor_SMD:R_0805_2012Metric_Pad1.20x1.40mm_HandSolder, F.Cu at (167.8, 69.1)
- added RFBVDD_VEE2: 10K, Resistor_SMD:R_0805_2012Metric_Pad1.20x1.40mm_HandSolder, F.Cu at (167.5, 94.5)
- added RFBVDD_VEE3: 10K, Resistor_SMD:R_0805_2012Metric_Pad1.20x1.40mm_HandSolder, F.Cu at (167.4, 122.2)
- added RFBVDD_VEE4: 10K, Resistor_SMD:R_0805_2012Metric_Pad1.20x1.40mm_HandSolder, F.Cu at (167.3, 152.9)
- added RFBVEE_COM1: 60K, Resistor_SMD:R_0805_2012Metric_Pad1.20x1.40mm_HandSolder, F.Cu at (175.9, 72.8)
- added RFBVEE_COM2: 60K, Resistor_SMD:R_0805_2012Metric_Pad1.20x1.40mm_HandSolder, F.Cu at (172.1, 102.3)
- added RFBVEE_COM3: 60K, Resistor_SMD:R_0805_2012Metric_Pad1.20x1.40mm_HandSolder, F.Cu at (175.9, 126.5)
- added RFBVEE_COM4: 60K, Resistor_SMD:R_0805_2012Metric_Pad1.20x1.40mm_HandSolder, F.Cu at (171.6, 160.9)
- added RFBVEE_VEE1: 20K, Resistor_SMD:R_0805_2012Metric_Pad1.20x1.40mm_HandSolder, F.Cu at (173.7, 70.9)
- added RFBVEE_VEE2: 20K, Resistor_SMD:R_0805_2012Metric_Pad1.20x1.40mm_HandSolder, F.Cu at (172.1, 100.2)
- added RFBVEE_VEE3: 20K, Resistor_SMD:R_0805_2012Metric_Pad1.20x1.40mm_HandSolder, F.Cu at (173.7, 124.4)
- added RFBVEE_VEE4: 20K, Resistor_SMD:R_0805_2012Metric_Pad1.20x1.40mm_HandSolder, F.Cu at (171.5, 156.2)
- added RLIM1_1: 2K, Resistor_SMD:R_0805_2012Metric_Pad1.20x1.40mm_HandSolder, F.Cu at (172.5, 74.0)
- added RLIM1_2: 2K, Resistor_SMD:R_0805_2012Metric_Pad1.20x1.40mm_HandSolder, F.Cu at (175.0, 104.6)
- added RLIM1_3: 2K, Resistor_SMD:R_0805_2012Metric_Pad1.20x1.40mm_HandSolder, F.Cu at (171.7, 127.5)
- added RLIM1_4: 2K, Resistor_SMD:R_0805_2012Metric_Pad1.20x1.40mm_HandSolder, F.Cu at (175.0, 163.4)
- added RLIM2_1: 6K8, Resistor_SMD:R_0805_2012Metric_Pad1.20x1.40mm_HandSolder, F.Cu at (177.9, 78.4)
- added RLIM2_2: 6K8, Resistor_SMD:R_0805_2012Metric_Pad1.20x1.40mm_HandSolder, F.Cu at (181.3, 108.1)
- added RLIM2_3: 6K8, Resistor_SMD:R_0805_2012Metric_Pad1.20x1.40mm_HandSolder, F.Cu at (178.1, 132.4)
- added RLIM2_4: 6K8, Resistor_SMD:R_0805_2012Metric_Pad1.20x1.40mm_HandSolder, F.Cu at (180.8, 167.0)
- added Rpu1: 100K, Resistor_SMD:R_0805_2012Metric_Pad1.20x1.40mm_HandSolder, F.Cu at (152.8, 71.0)
- added Rpu2: 100K, Resistor_SMD:R_0805_2012Metric_Pad1.20x1.40mm_HandSolder, F.Cu at (152.9, 99.1)
- added Rpu3: 100K, Resistor_SMD:R_0805_2012Metric_Pad1.20x1.40mm_HandSolder, F.Cu at (153.2, 124.5)
- added Rpu4: 100K, Resistor_SMD:R_0805_2012Metric_Pad1.20x1.40mm_HandSolder, F.Cu at (153.2, 157.2)
- added U10: ~, ZeniteSolar:SSOP-36, F.Cu at (156.6, 98.8)
- added U11: ~, ZeniteSolar:SSOP-36, F.Cu at (156.5, 124.6)
- added U12: ~, ZeniteSolar:SSOP-36, F.Cu at (156.9, 157.4)
- COUT1: value 22uF -> 10uF
- C_VDDA2, C_VDDA4, C_VDDB2, C_VDDB4: value 10uF -> 100nF
- L1: value 12uH -> 15uH
- R1: value 470K -> 3K
- R2: value 27K -> 1K
- R3: value 1k -> 3K
- R5: value 3K4 -> 13K7
- R6: value 51k -> 1K
- U1, U8: value UCC21550 -> UCC21520
- U4: footprint Package_TO_SOT_SMD:SOT-23-6_Handsoldering -> ZeniteSolar:SOT-563
- U7: value LM7805 -> ~; footprint Package_TO_SOT_THT:TO-220-3_Vertical -> ZeniteSolar:SSOP-36
- U9: value Opamp_Quad -> TL084
- moved C8 81.9 mm to (119.5, 164.6), turned to 90 degrees
- moved C9 77.4 mm to (121.7, 164.6), turned to 90 degrees
- moved R3 75.9 mm to (128.1, 170.1), turned to 180 degrees
- moved R2 73.5 mm to (136.8, 168.2), turned to 90 degrees
- moved R1 72.5 mm to (134.4, 168.1), turned to -90 degrees
- moved R6 65.9 mm to (130.2, 172.1), turned to 0 degrees
- moved U9 65.0 mm to (128.0, 164.4), turned to 90 degrees
- moved U7 20.6 mm to (156.8, 70.9), turned to 0 degrees
- moved L1 20.5 mm to (122.7, 73.4), turned to 0 degrees
- moved C3 20.1 mm to (122.6, 75.3), turned to 180 degrees
- moved COUT1 19.3 mm to (126.0, 74.5), turned to 90 degrees
- moved U4 18.1 mm to (121.7, 77.7)
- moved J1 16.9 mm to (108.4, 76.5)
- moved C1 15.7 mm to (117.7, 78.1), turned to -90 degrees
- moved C2 15.6 mm to (115.4, 78.2), turned to -90 degrees
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Connections:
- net VDDA2 renamed VDD3
- net VDDB1 renamed VDD2
- net VDDB2 renamed VDD4
- A1 pad 17: unconnected-(A1-D2-Pad17) -> DIS1
- A1 pad 18: unconnected-(A1-D3-Pad18) -> DIS2
- A1 pad 20: PWM1 -> PWM2
- A1 pad 21: PWM2 -> PWM1
- A1 pad 9: unconnected-(A1-A0-Pad9) -> ADC0
- C1 pad 1: +24V -> +18V
- C2 pad 1: +24V -> +18V
- C8 pad 1: +5V -> 5V
- C9 pad 1: +5V -> 5V
- COUT1 pad 2: +18V -> 5V
- CSnb1 pad 2: VA -> COM1
- CSnb3 pad 2: VB -> COM3
- C_DIS2 pad 1: DIS1 -> DIS2
- C_DS1a1 pad 2: VA -> COM1
- C_DS1b1 pad 2: VA -> COM1
- C_DS2a1 pad 1: VA -> COM1
- C_DS2b1 pad 1: VA -> COM1
- C_DS3a1 pad 2: VB -> COM3
- C_DS3b1 pad 2: VB -> COM3
- C_DS4a1 pad 1: VB -> COM3
- C_DS4b1 pad 1: VB -> COM3
- C_VCCI​a1 pad 1: +5V -> 5V
- C_VCCI​a2 pad 1: +5V -> 5V
- C_VCCI​b1 pad 1: +5V -> 5V
- C_VCCI​b2 pad 1: +5V -> 5V
- C_VDDA1 pad 1: VDDA1 -> VDD1
- C_VDDA1 pad 2: VSSA1 -> VEE1
- C_VDDA2 pad 1: VDDA1 -> VDD1
- C_VDDA2 pad 2: VSSA1 -> VEE1
- C_VDDA3 pad 2: VSSA2 -> VEE3
- C_VDDA4 pad 2: VSSA2 -> VEE3
- C_VDDB1 pad 2: VSSB1 -> VEE2
- C_VDDB2 pad 2: VSSB1 -> VEE2
- C_VDDB3 pad 2: VSSB2 -> VEE4
- C_VDDB4 pad 2: VSSB2 -> VEE4
- DSnb2 pad 2: VA -> COM1
- DSnb4 pad 2: VB -> COM3
- J1 pad 1: +24V -> +18V
- L1 pad 2: +18V -> 5V
- Q1 pad 2: VA -> COM1
- Q1 pad 3: VA -> COM1
- Q2 pad 2: Vsh -> BAT-
- Q2 pad 3: Vsh -> BAT-
- Q2 pad 4: VA -> COM1
- Q3 pad 2: VB -> COM3
- Q3 pad 3: VB -> COM3
- Q4 pad 2: Vsh -> BAT-
- Q4 pad 3: Vsh -> BAT-
- Q4 pad 4: VB -> COM3
- R1 pad 1: +24V -> ADC0
- R1 pad 2: Net-(U4-EN) -> Net-(U9B--)
- R2 pad 1: Net-(U4-EN) -> Net-(U9B--)
- R2 pad 2: BAT- -> Vref
- R3 pad 1: BAT- -> Net-(U9B-+)
- R3 pad 2: Net-(U9A--) -> BAT-
- R4 pad 1: +18V -> 5V
- R6 pad 1: Net-(U9A--) -> Net-(U9B-+)
- R6 pad 2: Net-(U9B-+) -> Vout
- RSnb2 pad 1: VA -> COM1
- RSnb2b1 pad 1: VA -> COM1
- RSnb4 pad 1: VB -> COM3
- RSnb4b1 pad 1: VB -> COM3
- R_GS1 pad 1: VSSA1 -> COM1
- R_GS2 pad 1: VSSB1 -> BAT-
- R_GS3 pad 1: VSSB2 -> BAT-
- R_GS4 pad 1: VSSA2 -> COM3
- U1 pad 14: VSSA1 -> VEE1
- U1 pad 16: VDDA1 -> VDD1
- U1 pad 3: +5V -> 5V
- U1 pad 8: +5V -> 5V
- U1 pad 9: VSSB1 -> VEE2
- U4 pad 1: +24V -> +18V
- U4 pad 5: Net-(U4-EN) -> unconnected-(U4-EN-Pad5)
- U7 pad 1: +18V -> BAT-
- U7 pad 3: +5V -> unconnected-(U7-~{PG}-Pad3)
- U8 pad 14: VSSA2 -> VEE3
- U8 pad 3: +5V -> 5V
- U8 pad 5: DIS1 -> DIS2
- U8 pad 8: +5V -> 5V
- U8 pad 9: VSSB2 -> VEE4
- U9 pad 1: Net-(U9B-+) -> (no net)
- U9 pad 2: Net-(U9A--) -> (no net)
- U9 pad 3: Vsh -> (no net)
- U9 pad 4: +5V -> 5V
- U9 pad 7: DIS1 -> ADC0
Routing:
- net COM3: track 0.00 -> 422.4 mm, vias 0 -> 5
- net COM1: track 0.00 -> 303.7 mm, vias 0 -> 3
- net BAT-: track 569.1 -> 308.6 mm, vias 16 -> 19
- net VB: track 233.6 -> 0.00 mm, vias 1 -> 0
- net VA: track 218.9 -> 0.00 mm, vias 1 -> 0
- net Vsh: track 145.5 -> 0.00 mm, vias 2 -> 0
- net VEE1: track 0.00 -> 134.9 mm, vias 0 -> 2
- net VEE3: track 0.00 -> 120.0 mm, vias 0 -> 2
- net +5V: track 115.9 -> 0.00 mm, vias 24 -> 0
- net VEE4: track 0.00 -> 103.3 mm, vias 0 -> 2
- net VEE2: track 0.00 -> 94.6 mm, vias 0 -> 2
- net 5V: track 0.00 -> 77.3 mm, vias 0 -> 8
- net DIS2: track 0.00 -> 74.6 mm, vias 0 -> 4
- net VDD1: track 0.00 -> 73.8 mm, vias 0 -> 4
- net 3v3: track 71.8 -> 0.00 mm
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- added copper zone on F.Cu, net 5V
- removed copper zone on F.Cu, net +5V
