File: Hardware/AcionamentoMotor50A.kicad_sch (KiCad schematic)
At the start: 19 parts, among them J1 Conn_01x02, J2 Conn_01x02, U4 TPS543021, U7 LM7805

Commit message: 2026_07_09
Feitas simulações da corrente do gate e escolha de um novo gate driver
Parts:
- added HS2: Heatsink, symbol Mechanical:Heatsink
Changed lines of the file:
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@@
+	)
+	(symbol
+		(lib_id "Mechanical:Heatsink")
+		(at 102.87 125.73 0)
+		(unit 1)
+		(body_style 1)
+		(exclude_from_sim no)
+		(in_bom yes)
+		(on_board yes)
+		(in_pos_files yes)
+		(dnp no)
+		(fields_autoplaced yes)
+		(property "Reference" "HS2"
+			(at 106.68 122.5549 0)
+			(show_name no)
+			(do_not_autoplace no)
+			(effects
+				(font
+					(size 1.27 1.27)
+				)
+				(justify left)
+			)
+		)
+		(property "Value" "Heatsink"
+			(at 106.68 125.0949 0)
+			(show_name no)
+			(do_not_autoplace no)
+			(effects
+				(font
+					(size 1.27 1.27)
+				)
+				(justify left)
+			)
+		)
+		(property "Footprint" ""
+			(at 103.1748 125.73 0)
+			(hide yes)
+			(show_name no)
+			(do_not_autoplace no)
+			(effects
+				(font
+					(size 1.27 1.27)
+				)
+			)
+		)
+		(property "Datasheet" ""
+			(at 103.1748 125.73 0)
+			(hide yes)
+			(show_name no)
+			(do_not_autoplace no)
+			(effects
+				(font
+					(size 1.27 1.27)
+				)
+			)
+		)
+		(property "Description" "Heatsink"
+			(at 102.87 125.73 0)
+			(hide yes)
+			(show_name no)
+			(do_not_autoplace no)
+			(effects
+				(font
+					(size 1.27 1.27)
+				)
+			)
+		)
+		(instances
+			(project "AcionamentoMotor50A"
+				(path "/b145dbd1-3039-470e-a340-e1336fd0da53"
+					(reference "HS2")
+					(unit 1)
+				)
+			)
+		)
 	)
 	(symbol

Commit message: 2026_07_22
Finalizada a PCB para fazer na fresa do IFSC
Parts:
- removed C4, C6: 100nF, Capacitor_SMD:C_0805_2012Metric_Pad1.18x1.45mm_HandSolder, symbol Device:C
- removed C5, C7: 10uF, Capacitor_SMD:C_0805_2012Metric_Pad1.18x1.45mm_HandSolder, symbol Device:C
- removed HS1: Heatsink, ZeniteSolar:Heatsink_120mmx100mm_H70mm, symbol Mechanical:Heatsink
- removed HS2: Heatsink, symbol Mechanical:Heatsink
- removed R1: 470K, Resistor_SMD:R_0805_2012Metric_Pad1.20x1.40mm_HandSolder, symbol Device:R
- removed R2: 27K, Resistor_SMD:R_0805_2012Metric_Pad1.20x1.40mm_HandSolder, symbol Device:R
- removed U7: LM7805, Package_TO_SOT_THT:TO-220-3_Vertical, symbol Regulator_Linear:L7805
- added COUT2: 100nF, Capacitor_SMD:C_0805_2012Metric_Pad1.18x1.45mm_HandSolder, symbol Device:C
- COUT1: value 22uF -> 10uF
- L1: value 12uH -> 15uH
- R5: value 3K4 -> 13K7
- U4: footprint Package_TO_SOT_SMD:SOT-23-6_Handsoldering -> ZeniteSolar:SOT-563
Connections:
- net +24V is gone; now on net +18V: C1.1, C2.1, J1.1 (Pin_1), U4.1 (VIN)
- net +18V: no longer COUT1.2, L1.2, R4.1
- net +5V: now also COUT1.2, L1.2, R4.1, COUT2.2
- net GNDREF: now also COUT2.1
- net PWM1: now also A1.21 (D6); no longer A1.20 (D5)
- net PWM2: now also A1.20 (D5); no longer A1.21 (D6)
- net DIS1: now reaches A1.17 (D2)
- net DIS2: now reaches A1.18 (D3)
- net ADC0: now reaches A1.9 (A0)
Other:
- note added: "+18V do barramento do Barco Usar um KREx2"
- note added: "Barramento do barco 48V"
- note removed: "+24V Deve vir de uma bateria Usar um KREx2"
- note removed: "Barramento do barco"
- note removed: "Saída +18V"
- moved on the sheet: A1, COUT1, R4, R5
