File: Hardware/PonteH.kicad_sch (KiCad schematic)
At the start: 63 parts, among them Q1 IXFN420N10T, Q2 IXFN420N10T, Q3 IXFN420N10T, Q4 IXFN420N10T, U1 UCC21550, U8 UCC21550

Commit message: 2026_07_22
Finalizada a PCB para fazer na fresa do IFSC
Parts:
- removed R_Sh1: 0.001R, Resistor_THT:R_Axial_Power_L20.0mm_W6.4mm_P25.40mm, symbol Device:R
- added HS1: Heatsink, ZeniteSolar:Heatsink_120mmx100mm_H70mm, symbol Mechanical:Heatsink
- C_VDDA2, C_VDDA4, C_VDDB2, C_VDDB4: value 10uF -> 100nF
- U1, U8: value UCC21550 -> UCC21520
Connections:
- net Vsh is gone; now on net BAT-: Q2.2 (DS), Q2.3 (S), Q4.2 (DS), Q4.3 (S)
- net VDDA1 renamed VDD1
- net VDDA2 renamed VDD3
- net VDDB1 renamed VDD2
- net VDDB2 renamed VDD4
- net VSSA1 renamed VEE1
- net VEE1: no longer R_GS1.1
- net VSSA2 renamed VEE3
- net VEE3: no longer R_GS4.1
- net VSSB1 renamed VEE2
- net VEE2: no longer R_GS2.1
- net VSSB2 renamed VEE4
- net VEE4: no longer R_GS3.1
- new net COM1: R_GS1.1
- new net COM2: R_GS2.1
- new net COM3: R_GS4.1
- new net COM4: R_GS3.1
