File: Hardware/TensaoIsolada.kicad_sch (KiCad schematic)
At the start: 72 parts, among them U2 UCC34141-Q1, U3 UCC34141-Q1, U5 UCC34141-Q1, U6 UCC34141-Q1

Commit message: 2026_07_03
Continuidade do roteamento..

foram roteados os drivers
Connections:
- net GND_ISO1: no longer C_VEE4.2, C_VEEGD4.2, LBB4.1
- net GND_ISO4: now also C_VEE4.2, C_VEEGD4.2, LBB4.1
Changed lines of the file:
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@@
 			)
 		)
-		(property "Value" "GND_ISO1"
-			(at 237.49 157.48 0)
+		(property "Value" "GND_ISO4"
+			(at 240.03 153.6699 0)
 			(show_name no)
 			(do_not_autoplace no)
@@
 					(size 1.27 1.27)
 				)
+				(justify left)
 			)
 		)

Commit message: 2026_07_22
Finalizada a PCB para fazer na fresa do IFSC
Parts:
- removed C_ENA1, C_ENA2, C_ENA3, C_ENA4, C_IN1b1, C_IN2b1, C_IN3b1, C_IN4b1, C_PG1, C_PG2, C_PG3, C_PG4, C_VDD1b1, C_VDD2b1, C_VDD3b1, C_VDD4b1, C_VDDGD1, C_VDDGD2, C_VDDGD3, C_VDDGD4: 100nF, Capacitor_SMD:C_0805_2012Metric_Pad1.18x1.45mm_HandSolder, symbol Device:C
- removed C_FBVDD1, C_FBVDD2, C_FBVDD3, C_FBVDD4: 220pF, Capacitor_SMD:C_0805_2012Metric_Pad1.18x1.45mm_HandSolder, symbol Device:C
- removed C_FBVEE1, C_FBVEE2, C_FBVEE3, C_FBVEE4: 10pF, Capacitor_SMD:C_0805_2012Metric_Pad1.18x1.45mm_HandSolder, symbol Device:C
- removed C_IN1, C_IN2, C_IN3, C_IN4, C_VDD1, C_VDD2, C_VDD3, C_VDD4: 10uF, Capacitor_SMD:C_0805_2012Metric_Pad1.18x1.45mm_HandSolder, symbol Device:C
- removed C_VEE1, C_VEE2, C_VEE3, C_VEE4: 2,2uF, Capacitor_SMD:C_0805_2012Metric_Pad1.18x1.45mm_HandSolder, symbol Device:C
- removed C_VEEGD1, C_VEEGD2, C_VEEGD3, C_VEEGD4: 6,8uF, Capacitor_SMD:C_0805_2012Metric_Pad1.18x1.45mm_HandSolder, symbol Device:C
- removed LBB1, LBB2, LBB3, LBB4: 3,3uH, Inductor_SMD:L_0805_2012Metric_Pad1.05x1.20mm_HandSolder, symbol Device:L
- removed R_ENA1, R_ENA2, R_ENA3, R_ENA4, R_PG1, R_PG2, R_PG3, R_PG4: 5K1, Resistor_SMD:R_0805_2012Metric_Pad1.20x1.40mm_HandSolder, symbol Device:R
- removed R_FBVDDBOT1, R_FBVDDBOT2, R_FBVDDBOT3, R_FBVDDBOT4: 10K, Resistor_SMD:R_0805_2012Metric_Pad1.20x1.40mm_HandSolder, symbol Device:R
- removed R_FBVDDTOP1, R_FBVDDTOP2, R_FBVDDTOP3, R_FBVDDTOP4: 50K, Resistor_SMD:R_0805_2012Metric_Pad1.20x1.40mm_HandSolder, symbol Device:R
- removed R_FBVEE1, R_FBVEE2, R_FBVEE3, R_FBVEE4: 55K, Resistor_SMD:R_0805_2012Metric_Pad1.20x1.40mm_HandSolder, symbol Device:R
- removed U2, U3, U5, U6: UCC34141-Q1, ZeniteSolar:SSOP-16_4.55x10.63mm_P0.65mm, symbol ZeniteSolar:UCC34141-Q1
- added CFBVDD_1, CFBVDD_2, CFBVDD_3, CFBVDD_4, CFBVEE_1, CFBVEE_2, CFBVEE_3, CFBVEE_4: 330pF, Capacitor_SMD:C_0805_2012Metric_Pad1.18x1.45mm_HandSolder, symbol Device:C
- added Cin1, Cin2, Cin3, Cin4: 20uF, Capacitor_SMD:C_0805_2012Metric_Pad1.18x1.45mm_HandSolder, symbol Device:C
- added Cin1b1, Cin2b1, Cin3b1, Cin4b1, Cout1a1, Cout2a1, Cout3a1, Cout4a1: 100nF, Capacitor_SMD:C_0805_2012Metric_Pad1.18x1.45mm_HandSolder, symbol Device:C
- added Cout1b1, Cout1c1, Cout2b1, Cout2c1, Cout3b1, Cout3c1, Cout4b1, Cout4c1: 10uF, Capacitor_SMD:C_0805_2012Metric_Pad1.18x1.45mm_HandSolder, symbol Device:C
- added Cout2_1, Cout2_2, Cout2_3, Cout2_4: 4.7uF, Capacitor_SMD:C_0805_2012Metric_Pad1.18x1.45mm_HandSolder, symbol Device:C
- added Cout3_1, Cout3_2, Cout3_3, Cout3_4: 12uF, Capacitor_SMD:C_0805_2012Metric_Pad1.18x1.45mm_HandSolder, symbol Device:C
- added D1, D2, D3, D4: 1N4148, Diode_THT:D_DO-35_SOD27_P7.62mm_Horizontal, symbol Device:D
- added RFBVDD_VDD1, RFBVDD_VDD2, RFBVDD_VDD3, RFBVDD_VDD4: 90K, Resistor_SMD:R_0805_2012Metric_Pad1.20x1.40mm_HandSolder, symbol Device:R
- added RFBVDD_VEE1, RFBVDD_VEE2, RFBVDD_VEE3, RFBVDD_VEE4: 10K, Resistor_SMD:R_0805_2012Metric_Pad1.20x1.40mm_HandSolder, symbol Device:R
- added RFBVEE_COM1, RFBVEE_COM2, RFBVEE_COM3, RFBVEE_COM4: 60K, Resistor_SMD:R_0805_2012Metric_Pad1.20x1.40mm_HandSolder, symbol Device:R
- added RFBVEE_VEE1, RFBVEE_VEE2, RFBVEE_VEE3, RFBVEE_VEE4: 20K, Resistor_SMD:R_0805_2012Metric_Pad1.20x1.40mm_HandSolder, symbol Device:R
- added RLIM1_1, RLIM1_2, RLIM1_3, RLIM1_4: 2K, Resistor_SMD:R_0805_2012Metric_Pad1.20x1.40mm_HandSolder, symbol Device:R
- added RLIM2_1, RLIM2_2, RLIM2_3, RLIM2_4: 6K8, Resistor_SMD:R_0805_2012Metric_Pad1.20x1.40mm_HandSolder, symbol Device:R
- added Rpu1, Rpu2, Rpu3, Rpu4: 100K, Resistor_SMD:R_0805_2012Metric_Pad1.20x1.40mm_HandSolder, symbol Device:R
- added U10, U11, U12, U7: (no value), ZeniteSolar:SSOP-36, symbol ZeniteSolar:UCC14341-Q1
Connections:
- net +18V: now also Cin1.1, Cin1b1.1, Cin2.1, Cin2b1.1, Cin3.1, Cin3b1.1, Cin4.1, Cin4b1.1, U10.6 (VIN), U10.7 (VIN), U11.6 (VIN), U11.7 (VIN), U12.6 (VIN), U12.7 (VIN), U7.6 (VIN), U7.7 (VIN)
- net +5V: now also Rpu1.1, Rpu2.1, Rpu3.1, Rpu4.1
- net FBVDD2: now also CFBVDD_2.1, RFBVDD_VDD2.1, RFBVDD_VEE2.1, U10.34 (FBVDD)
- net FBVDD3: now also CFBVDD_3.1, RFBVDD_VDD3.1, RFBVDD_VEE3.1, U11.34 (FBVDD)
- net FBVDD4: now also CFBVDD_4.1, RFBVDD_VDD4.1, RFBVDD_VEE4.1, U12.34 (FBVDD)
- net FBVEE2: now also CFBVEE_2.1, RFBVEE_COM2.1, RFBVEE_VEE2.1, U10.33 (FBVEE)
- net FBVEE3: now also CFBVEE_3.1, RFBVEE_COM3.1, RFBVEE_VEE3.1, U11.33 (FBVEE)
- net FBVEE4: now also CFBVEE_4.1, RFBVEE_COM4.1, RFBVEE_VEE4.1, U12.33 (FBVEE)
- net GNDREF: now also Cin1.2, Cin1b1.2, Cin2.2, Cin2b1.2, Cin3.2, Cin3b1.2, Cin4.2, Cin4b1.2, U10.1 (GNDP), U10.10 (GNDP), U10.11 (GNDP), U10.12 (GNDP), U10.13 (GNDP), U10.14 (GNDP), U10.15 (GNDP), U10.16 (GNDP), U10.17 (GNDP), U10.18 (GNDP), U10.2 (GNDP), U10.5 (GNDP), U10.8 (GNDP), U10.9 (GNDP), U11.1 (GNDP), U11.10 (GNDP), U11.11 (GNDP), U11.12 (GNDP), U11.13 (GNDP), U11.14 (GNDP), U11.15 (GNDP), U11.16 (GNDP), U11.17 (GNDP), U11.18 (GNDP), U11.2 (GNDP), U11.5 (GNDP), U11.8 (GNDP), U11.9 (GNDP), U12.1 (GNDP), U12.10 (GNDP), U12.11 (GNDP), U12.12 (GNDP), U12.13 (GNDP), U12.14 (GNDP), U12.15 (GNDP), U12.16 (GNDP), U12.17 (GNDP), U12.18 (GNDP), U12.2 (GNDP), U12.5 (GNDP), U12.8 (GNDP), U12.9 (GNDP), U7.1 (GNDP), U7.10 (GNDP), U7.11 (GNDP), U7.12 (GNDP), U7.13 (GNDP), U7.14 (GNDP), U7.15 (GNDP), U7.16 (GNDP), U7.17 (GNDP), U7.18 (GNDP), U7.2 (GNDP), U7.5 (GNDP), U7.8 (GNDP), U7.9 (GNDP)
- net GND_ISO1: now also Cout2_1.2, Cout3_1.2, RFBVEE_COM1.2, RLIM1_1.1, RLIM2_1.2
- net GND_ISO2: now also Cout2_2.2, Cout2_4.2, Cout3_2.2, Cout3_4.2, RFBVEE_COM2.2, RFBVEE_COM4.2, RLIM1_2.1, RLIM1_4.1, RLIM2_2.2, RLIM2_4.2
- net GND_ISO3: now also Cout2_3.2, Cout3_3.2, RFBVEE_COM3.2, RLIM1_3.1, RLIM2_3.2
- new net: D4.2 (A), RLIM2_4.1
- new net: Rpu4.2, U12.4 (ENA)
- new net: Rpu3.2, U11.4 (ENA)
- new net: D3.2 (A), RLIM2_3.1
- new net: D1.2 (A), RLIM2_1.1
- new net: D2.2 (A), RLIM2_2.1
- new net: Rpu1.2, U7.4 (ENA)
- new net: Rpu2.2, U10.4 (ENA)
- new net +15_ISO1: Cout1a1.1, Cout1b1.1, Cout1c1.1, Cout2_1.1, RFBVDD_VDD1.2, U7.28 (VDD), U7.29 (VDD)
- new net +15_ISO2: Cout2_2.1, Cout2a1.1, Cout2b1.1, Cout2c1.1, RFBVDD_VDD2.2, U10.28 (VDD), U10.29 (VDD)
- new net +15_ISO3: Cout2_3.1, Cout3a1.1, Cout3b1.1, Cout3c1.1, RFBVDD_VDD3.2, U11.28 (VDD), U11.29 (VDD)
- new net +15_ISO4: Cout2_4.1, Cout4a1.1, Cout4b1.1, Cout4c1.1, RFBVDD_VDD4.2, U12.28 (VDD), U12.29 (VDD)
- new net -10_ISO1: CFBVDD_1.2, CFBVEE_1.2, Cout1a1.2, Cout1b1.2, Cout1c1.2, Cout3_1.1, RFBVDD_VEE1.2, RFBVEE_VEE1.2, U7.19 (VEE), U7.20 (VEE), U7.21 (VEE), U7.22 (VEE), U7.23 (VEE), U7.24 (VEE), U7.25 (VEE), U7.26 (VEE), U7.27 (VEE), U7.30 (VEE), U7.31 (VEE), U7.35 (VEEA), U7.36 (VEE)
- new net -10_ISO2: CFBVDD_2.2, CFBVEE_2.2, Cout2a1.2, Cout2b1.2, Cout2c1.2, Cout3_2.1, RFBVDD_VEE2.2, RFBVEE_VEE2.2, U10.19 (VEE), U10.20 (VEE), U10.21 (VEE), U10.22 (VEE), U10.23 (VEE), U10.24 (VEE), U10.25 (VEE), U10.26 (VEE), U10.27 (VEE), U10.30 (VEE), U10.31 (VEE), U10.35 (VEEA), U10.36 (VEE)
- new net -10_ISO3: CFBVDD_3.2, CFBVEE_3.2, Cout3_3.1, Cout3a1.2, Cout3b1.2, Cout3c1.2, RFBVDD_VEE3.2, RFBVEE_VEE3.2, U11.19 (VEE), U11.20 (VEE), U11.21 (VEE), U11.22 (VEE), U11.23 (VEE), U11.24 (VEE), U11.25 (VEE), U11.26 (VEE), U11.27 (VEE), U11.30 (VEE), U11.31 (VEE), U11.35 (VEEA), U11.36 (VEE)
- new net -10_ISO4: CFBVDD_4.2, CFBVEE_4.2, Cout3_4.1, Cout4a1.2, Cout4b1.2, Cout4c1.2, RFBVDD_VEE4.2, RFBVEE_VEE4.2, U12.19 (VEE), U12.20 (VEE), U12.21 (VEE), U12.22 (VEE), U12.23 (VEE), U12.24 (VEE), U12.25 (VEE), U12.26 (VEE), U12.27 (VEE), U12.30 (VEE), U12.31 (VEE), U12.35 (VEEA), U12.36 (VEE)
- new net FBVDD1: CFBVDD_1.1, RFBVDD_VDD1.1, RFBVDD_VEE1.1, U7.34 (FBVDD)
- new net FBVEE1: CFBVEE_1.1, RFBVEE_COM1.1, RFBVEE_VEE1.1, U7.33 (FBVEE)
- new net RLIM1: D1.1 (K), RLIM1_1.2, U7.32 (RLIM)
- new net RLIM2: D2.1 (K), RLIM1_2.2, U10.32 (RLIM)
- new net RLIM3: D3.1 (K), RLIM1_3.2, U11.32 (RLIM)
- new net RLIM4: D4.1 (K), RLIM1_4.2, U12.32 (RLIM)
Other:
- note added: "Tensão Isolada 1"
- note added: "Tensão Isolada 2"
- note added: "Tensão Isolada 3"
- note added: "Tensão Isolada 4"
- note removed: "Tensão isolada 1"
- note removed: "Tensão isolada 2"
- note removed: "Tensão isolada 3"
- note removed: "Tensão isolada 4"
